File: 555-timer-pwm-with-digipot/555-timer-pwm-with-digipot.kicad_sch (KiCad schematic)
At the start: 19 parts, among them J1 Conn_01x05_Pin

Commit message: Add footprints for 555 timer.
555 timer needed custom footprint. Downloaded model off the internet
somewhere.

The digipot seems to fit the MSOP-10_3x3mm_P0.5mm footprint and model
from preloaded library.
Parts:
- C1, C2, C3, C4: footprint (none) -> Capacitor_SMD:C_0805_2012Metric
- D1, D2: footprint Diode_THT:D_DO-35_SOD27_P7.62mm_Horizontal -> Diode_SMD:D_SOD-123
- J1: footprint (none) -> Connector_PinHeader_2.54mm:PinHeader_1x05_P2.54mm_Vertical
- JP1, JP2: footprint (none) -> Jumper:SolderJumper-2_P1.3mm_Open_TrianglePad1.0x1.5mm
- R1, R2, R3, R4, R5: footprint (none) -> Resistor_SMD:R_0805_2012Metric
- TP1, TP2, TP3: footprint (none) -> TestPoint:TestPoint_THTPad_D2.0mm_Drill1.0mm
- U1: footprint (none) -> project:SOIC-8_3.9x4.9mm_P1.27mm
- U2: footprint (none) -> Package_SO:MSOP-10_3x3mm_P0.5mm
Changed lines of the file:
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@@
       (effects (font (size 1.27 1.27)) (justify right))
     )
-    (property "Footprint" "" (at 148.59 110.49 0)
+    (property "Footprint" "TestPoint:TestPoint_THTPad_D2.0mm_Drill1.0mm" (at 148.59 110.49 0)
       (effects (font (size 1.27 1.27)) hide)
     )
@@
       (effects (font (size 1.27 1.27)) (justify left))
     )
-    (property "Footprint" "Diode_THT:D_DO-35_SOD27_P7.62mm_Horizontal" (at 147.955 87.63 0)
+    (property "Footprint" "Diode_SMD:D_SOD-123" (at 147.955 87.63 0)
       (effects (font (size 1.27 1.27)) hide)
     )
@@
       (effects (font (size 1.27 1.27)) (justify left))
     )
-    (property "Footprint" "" (at 145.7452 123.19 0)
+    (property "Footprint" "Capacitor_SMD:C_0805_2012Metric" (at 145.7452 123.19 0)
       (effects (font (size 1.27 1.27)) hide)
     )
@@
       (effects (font (size 1.27 1.27)))
     )
-    (property "Footprint" "" (at 176.53 52.07 0)
+    (property "Footprint" "Connector_PinHeader_2.54mm:PinHeader_1x05_P2.54mm_Vertical" (at 176.53 52.07 0)
       (effects (font (size 1.27 1.27)) hide)
     )
@@
       (effects (font (size 1.27 1.27)) (justify left))
     )
-    (property "Footprint" "" (at 160.02 53.34 0)
+    (property "Footprint" "Jumper:SolderJumper-2_P1.3mm_Open_TrianglePad1.0x1.5mm" (at 160.02 53.34 0)
       (effects (font (size 1.27 1.27)) hide)
     )
@@
       (effects (font (size 1.27 1.27)) (justify left))
     )
-    (property "Footprint" "" (at 122.682 53.34 90)
+    (property "Footprint" "Resistor_SMD:R_0805_2012Metric" (at 122.682 53.34 90)
       (effects (font (size 1.27 1.27)) hide)
     )
@@
       (effects (font (size 1.27 1.27)) (justify left))
     )
-    (property "Footprint" "" (at 98.552 120.65 90)
+    (property "Footprint" "Resistor_SMD:R_0805_2012Metric" (at 98.552 120.65 90)
       (effects (font (size 1.27 1.27)) hide)
     )
@@
       (effects (font (size 1.27 1.27)))
     )
-    (property "Footprint" "" (at 110.49 99.06 0)
+    (property "Footprint" "Package_SO:MSOP-10_3x3mm_P0.5mm" (at 110.49 99.06 0)
       (effects (font (size 1.27 1.27)) hide)
     )
@@
       (effects (font (size 1.27 1.27)))
     )
-    (property "Footprint" "" (at 149.86 93.98 0)
+    (property "Footprint" "TestPoint:TestPoint_THTPad_D2.0mm_Drill1.0mm" (at 149.86 93.98 0)
       (effects (font (size 1.27 1.27)) hide)
     )
@@
       (effects (font (size 1.27 1.27)) (justify left))
     )
-    (property "Footprint" "" (at 143.002 77.47 90)
+    (property "Footprint" "Resistor_SMD:R_0805_2012Metric" (at 143.002 77.47 90)
       (effects (font (size 1.27 1.27)) hide)
     )
@@
       (effects (font (size 1.27 1.27)) (justify left))
     )
-    (property "Footprint" "" (at 194.0052 97.79 0)
+    (property "Footprint" "Capacitor_SMD:C_0805_2012Metric" (at 194.0052 97.79 0)
       (effects (font (size 1.27 1.27)) hide)
     )
@@
       (effects (font (size 1.27 1.27)) (justify right))
     )
-    (property "Footprint" "Diode_THT:D_DO-35_SOD27_P7.62mm_Horizontal" (at 141.605 87.63 0)
+    (property "Footprint" "Diode_SMD:D_SOD-123" (at 141.605 87.63 0)
       (effects (font (size 1.27 1.27)) hide)
     )
@@
       (effects (font (size 1.27 1.27)) (justify left))
     )
-    (property "Footprint" "" (at 131.7752 123.19 0)
+    (property "Footprint" "Capacitor_SMD:C_0805_2012Metric" (at 131.7752 123.19 0)
       (effects (font (size 1.27 1.27)) hide)
     )
@@
       (effects (font (size 1.27 1.27)) (justify left))
     )
-    (property "Footprint" "" (at 132.842 53.34 90)
+    (property "Footprint" "Resistor_SMD:R_0805_2012Metric" (at 132.842 53.34 90)
       (effects (font (size 1.27 1.27)) hide)
     )
@@
       (effects (font (size 1.27 1.27)) (justify left))
     )
-    (property "Footprint" "" (at 82.8548 115.57 0)
+    (property "Footprint" "Capacitor_SMD:C_0805_2012Metric" (at 82.8548 115.57 0)
       (effects (font (size 1.27 1.27)) hide)
     )
@@
       (effects (font (size 1.27 1.27)) (justify left))
     )
-    (property "Footprint" "" (at 89.662 120.65 90)
+    (property "Footprint" "Resistor_SMD:R_0805_2012Metric" (at 89.662 120.65 90)
       (effects (font (size 1.27 1.27)) hide)
     )
@@
       (effects (font (size 1.27 1.27)))
     )
-    (property "Footprint" "" (at 168.91 105.41 0)
+    (property "Footprint" "project:SOIC-8_3.9x4.9mm_P1.27mm" (at 168.91 105.41 0)
       (effects (font (size 1.27 1.27)) hide)
     )
@@
       (effects (font (size 1.27 1.27)))
     )
-    (property "Footprint" "" (at 134.62 93.98 0)
+    (property "Footprint" "TestPoint:TestPoint_THTPad_D2.0mm_Drill1.0mm" (at 134.62 93.98 0)
       (effects (font (size 1.27 1.27)) hide)
     )
@@
       (effects (font (size 1.27 1.27)) (justify left))
     )
-    (property "Footprint" "" (at 152.4 53.34 0)
-      (effects (font (size 1.27 1.27)) hide)
-    )
+    (property "Footprint" "Jumper:SolderJumper-2_P1.3mm_Open_TrianglePad1.0x1.5mm" (at 152.4 53.34 0)
+      (effects (font (size 1.27 1.27)) hide)
+    )
