File: mipi-dsi-breakout/lcd-side-interface/lcd-side-interface.kicad_pcb (KiCad board)
At the start: 2 copper layers, 60 x 63.5 mm, 9 parts

Commit message: Flip orientation of 40pin zif pads.
The connector footprint is on the wrong side (cable goes in the opposite
side of the lever). Flip the pads to original orientation to match
part...

Add user drawings annotation and measurements to lcd side pcb.
Parts:
- moved et050fw04_t_dsi1 19.7 mm to (162.5, 78.5), turned to -90 degrees
Other:
- board text added: "middle line"

Commit message: Correct orientation & position of zif connectors.
Parts:
- moved tst050hdbs_80c_dsi1 8.56 mm to (137.0, 73.8), turned to -90 degrees
- moved tst043wvbi_130c_ctp1 6.65 mm to (142.7, 81.0), turned to -90 degrees
- moved tst043wvbi_130c_dsi1 6.32 mm to (155.0, 110.5)
- moved et060hd02_t_dsi1 4.72 mm to (130.9, 84.0), turned to -90 degrees
- moved tst050hdbs_80c_ctp1 4.12 mm to (138.5, 99.2), turned to -90 degrees
- moved H1 3.00 mm to (130.5, 110.0)
- moved JP1 2.00 mm to (172.0, 117.5)
Routing:
- net /RESET: track 3.85 -> 0.01 mm
